Commit message: changes to drive to enhance smoother turning and terrain navigation

File: urdf/rocker_bogie_rover_final.urdf (robot description, URDF)
Before this commit: robot rocker_bogie_rover_final, 11 links, 10 joints
Joints:
- joint joint_wheel_fl: limit (none) -> effort=50.0 velocity=10.0
- joint joint_wheel_fr: limit (none) -> effort=50.0 velocity=10.0
- joint joint_wheel_ml: limit (none) -> effort=50.0 velocity=10.0
- joint joint_wheel_mr: limit (none) -> effort=50.0 velocity=10.0
- joint joint_wheel_rl: limit (none) -> effort=50.0 velocity=10.0
- joint joint_wheel_rr: limit (none) -> effort=50.0 velocity=10.0

File: urdf/rocker_bogie_rover_visual.urdf (robot description, URDF)
Before this commit: robot rocker_bogie_rover_visual, 16 links, 15 joints
Joints:
- joint joint_wheel_fl: limit (none) -> effort=50.0 velocity=10.0
- joint joint_wheel_fr: limit (none) -> effort=50.0 velocity=10.0
- joint joint_wheel_ml: limit (none) -> effort=50.0 velocity=10.0
- joint joint_wheel_mr: limit (none) -> effort=50.0 velocity=10.0
- joint joint_wheel_rl: limit (none) -> effort=50.0 velocity=10.0
- joint joint_wheel_rr: limit (none) -> effort=50.0 velocity=10.0
