Commit message: Lidar sensor added

File: urdf/rocker_bogie_rover_visual.urdf (robot description, URDF)
Before this commit: robot rocker_bogie_rover_visual, 14 links, 13 joints
Links:
- added link lidar_link, mass 0.15; collision cylinder length=0.06 radius=0.05; visual cylinder length=0.06 radius=0.05
Joints:
- added joint lidar_joint: type fixed, parent base_link, child lidar_link, origin xyz=0 0 0.30 rpy=0 0 0

Commit message: TF tree stablized, robot model visible in Rviz, LIDAR scan working

File: urdf/rocker_bogie_rover_visual.urdf (robot description, URDF)
Before this commit: robot rocker_bogie_rover_visual, 15 links, 14 joints
Links:
- added link imu_link, mass 0.05; collision box size=0.04 0.04 0.02; visual box size=0.04 0.04 0.02
Joints:
- added joint imu_joint: type fixed, parent base_link, child imu_link, origin xyz=0 0 0.12 rpy=0 0 0

Commit message: fix(urdf): tune skid-steer friction and joint limits for smoother turning
Reduced lateral friction (mu2) and added fdir1 properly to wheel joints. Increased velocity and effort limits extensively across all wheels to overcome static turning impedance. Tweaked diff drive plugin max angular acceleration to improve steering responsiveness.

File: urdf/rocker_bogie_rover_visual.urdf (robot description, URDF)
Before this commit: robot rocker_bogie_rover_visual, 16 links, 15 joints
Joints:
- joint joint_wheel_fl: limit effort=50.0 velocity=10.0 -> effort=400.0 velocity=30.0
- joint joint_wheel_fr: limit effort=50.0 velocity=10.0 -> effort=400.0 velocity=30.0
- joint joint_wheel_ml: limit effort=50.0 velocity=10.0 -> effort=400.0 velocity=30.0
- joint joint_wheel_mr: limit effort=50.0 velocity=10.0 -> effort=400.0 velocity=30.0
- joint joint_wheel_rl: limit effort=50.0 velocity=10.0 -> effort=400.0 velocity=30.0
- joint joint_wheel_rr: limit effort=50.0 velocity=10.0 -> effort=400.0 velocity=30.0
